File: build-system/erbui/generators/front_pcb/alpha.9mm/alpha.9mm.wire.kicad_pcb (KiCad board)
At the start: 2 copper layers, 1 part

Commit message: Update pcbs
Parts:
- added ZZ1: 100k, Potentiometer_Thonk:AlphaPot9ShaftD, F.Cu at (0.00, 0.00)
Changed lines of the file:
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@@
     (tracks 2)
     (zones 0)
-    (modules 1)
-    (nets 2)
+    (modules 2)
+    (nets 4)
   )
   (page A4)
@@
   )
   (net 0 "")
-  (net 1 "Net-(Pin0-Pad1)")
+  (net 1 +3V3)
+  (net 2 GND)
+  (net 3 "Net-(Pin0-Pad1)")
   (net_class Default "This is the default net class."
     (clearance 0.1524)
@@
     (diff_pair_width 0.1524)
     (diff_pair_gap 0.1524)
+    (add_net +3V3)
+    (add_net GND)
     (add_net "Net-(Pin0-Pad1)")
+  )
+  (module Potentiometer_Thonk:AlphaPot9ShaftD locked (layer F.Cu)
+    (at 0 0)
+    (fp_text reference ZZ1 (at 0 4.7) (layer F.SilkS) hide
+      (effects (font (size 1 1) (thickness 0.15)))
+    )
+    (fp_text value 100k (at 0 10.1) (layer F.Fab)
+      (effects (font (size 1 1) (thickness 0.15)))
+    )
+    (fp_circle (center -3.8 5.6) (end -4.2 5.6) (layer F.SilkS) (width 0.15))
+    (fp_circle (center 3.8 -3.8) (end 4.2 -3.8) (layer F.SilkS) (width 0.15))
+    (fp_line (start -2.6 1.5) (end 2.6 1.5) (layer F.SilkS) (width 0.15))
+    (fp_circle (center 0 0) (end 3 0) (layer F.SilkS) (width 0.15))
+    (fp_line (start 3.7 6.5) (end 4.7 6.5) (layer F.SilkS) (width 0.15))
+    (fp_line (start 4.7 1.4) (end 4.7 6.5) (layer F.SilkS) (width 0.15))
+    (fp_line (start -4.7 1.4) (end -4.7 6.5) (layer F.SilkS) (width 0.15))
+    (fp_line (start -4.7 6.5) (end -3.7 6.5) (layer F.SilkS) (width 0.15))
+    (fp_line (start -4.7 -4.8) (end -4.7 -1.4) (layer F.SilkS) (width 0.15))
+    (fp_line (start 4.7 -4.8) (end 4.7 -1.4) (layer F.SilkS) (width 0.15))
+    (fp_line (start -4.7 -4.8) (end 4.7 -4.8) (layer F.SilkS) (width 0.15))
+    (fp_arc (start 0 0) (end -1.6 1.5) (angle 265) (layer F.SilkS) (width 0.15))
+    (pad "" thru_hole oval (at 5.7 0) (size 2.5 1.8) (drill oval 1.8 1.1) (layers *.Cu *.Mask))
+    (pad 3 thru_hole oval (at 2.5 7.5) (size 1.7 1.7) (drill 1) (layers *.Cu *.Mask)
+      (net 1 +3V3))
+    (pad 2 thru_hole oval (at 0 7.5) (size 1.7 1.7) (drill 1) (layers *.Cu *.Mask)
+      (net 3 "Net-(Pin0-Pad1)"))
+    (pad 1 thru_hole oval (at -2.5 7.5) (size 1.7 1.7) (drill 1) (layers *.Cu *.Mask)
+      (net 2 GND))
+    (pad "" thru_hole oval (at -5.7 0) (size 2.5 1.8) (drill oval 1.8 1.1) (layers *.Cu *.Mask))
   )
   (module TestPoint:TestPoint_Pad_D1.5mm (layer B.Cu)
@@
       (effects (font (size 1 1) (thickness 0.15)) (justify mirror))
     )
+    (fp_circle (center 0 0) (end 0 -0.95) (layer B.SilkS) (width 0.12))
     (fp_circle (center 0 0) (end 1.25 0) (layer B.CrtYd) (width 0.05))
-    (fp_circle (center 0 0) (end 0 -0.95) (layer B.SilkS) (width 0.12))
     (fp_text user %R (at 0 1.65) (layer B.Fab)
       (effects (font (size 1 1) (thickness 0.15)) (justify mirror))
     )
     (pad 1 smd circle (at 0 0) (size 1.5 1.5) (layers B.Cu B.Mask)
-      (net 1 "Net-(Pin0-Pad1)"))
+      (net 3 "Net-(Pin0-Pad1)"))
   )
   (gr_text pin (at -1.016 4.445) (layer B.SilkS)
     (effects (font (size 1 1) (thickness 0.15)) (justify left mirror))
   )
-  (segment (start 0 7.5) (end 0 7.62) (width 0.635) (layer B.Cu) (net 1))
-  (segment (start 0 7.62) (end 0 4.445) (width 0.635) (layer B.Cu) (net 1))
+  (segment (start 0 7.5) (end 0 7.62) (width 0.635) (layer B.Cu) (net 3))
+  (segment (start 0 7.62) (end 0 4.445) (width 0.635) (layer B.Cu) (net 3))
 )
