File: build-system/erbui/generators/front_pcb/led.3mm.rgb/led.3mm.rgb.wire.kicad_pcb (KiCad board)
At the start: 2 copper layers, 3 parts

Commit message: Update pcbs
Parts:
- added ZZ1: LED_RGBA, LED_SMD:LED_Cree-PLCC4_3.2x2.8mm_CCW, F.Cu at (0.00, 0.00)
Changed lines of the file:
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@@
     (tracks 13)
     (zones 0)
-    (modules 3)
-    (nets 4)
+    (modules 4)
+    (nets 5)
   )
   (page A4)
@@
   )
   (net 0 "")
-  (net 1 "Net-(Pin0-Pad1)")
-  (net 2 "Net-(Pin1-Pad1)")
-  (net 3 "Net-(Pin2-Pad1)")
+  (net 1 +3V3)
+  (net 2 "Net-(Pin0-Pad1)")
+  (net 3 "Net-(Pin1-Pad1)")
+  (net 4 "Net-(Pin2-Pad1)")
   (net_class Default "This is the default net class."
     (clearance 0.1524)
@@
     (diff_pair_width 0.1524)
     (diff_pair_gap 0.1524)
+    (add_net +3V3)
     (add_net "Net-(Pin0-Pad1)")
     (add_net "Net-(Pin1-Pad1)")
@@
       (effects (font (size 1 1) (thickness 0.15)) (justify mirror))
     )
+    (fp_circle (center 0 0) (end 1.25 0) (layer B.CrtYd) (width 0.05))
     (fp_circle (center 0 0) (end 0 -0.95) (layer B.SilkS) (width 0.12))
-    (fp_circle (center 0 0) (end 1.25 0) (layer B.CrtYd) (width 0.05))
     (fp_text user %R (at 0 1.65) (layer B.Fab)
       (effects (font (size 1 1) (thickness 0.15)) (justify mirror))
     )
     (pad 1 smd circle (at 0 0) (size 1.5 1.5) (layers B.Cu B.Mask)
-      (net 1 "Net-(Pin0-Pad1)"))
+      (net 2 "Net-(Pin0-Pad1)"))
+  )
+  (module LED_SMD:LED_Cree-PLCC4_3.2x2.8mm_CCW locked (layer F.Cu)
+    (at 0 0)
+    (descr "3.2mm x 2.8mm PLCC4 LED, http://www.cree.com/led-components/media/documents/CLV1AFKB(874).pdf")
+    (tags "LED Cree PLCC-4")
+    (attr smd)
+    (fp_text reference ZZ1 (at 0 -2.65) (layer F.SilkS) hide
+      (effects (font (size 1 1) (thickness 0.15)))
+    )
+    (fp_text value LED_RGBA (at 0 2.65) (layer F.Fab)
+      (effects (font (size 1 1) (thickness 0.15)))
+    )
+    (fp_circle (center 0 0) (end 1.12 0) (layer F.Fab) (width 0.1))
+    (fp_line (start -2.2 -1.75) (end -2.2 1.75) (layer F.CrtYd) (width 0.05))
+    (fp_line (start -2.2 1.75) (end 2.2 1.75) (layer F.CrtYd) (width 0.05))
+    (fp_line (start 2.2 1.75) (end 2.2 -1.75) (layer F.CrtYd) (width 0.05))
+    (fp_line (start 2.2 -1.75) (end -2.2 -1.75) (layer F.CrtYd) (width 0.05))
+    (fp_line (start -0.6 -1.4) (end -1.6 -0.4) (layer F.Fab) (width 0.1))
+    (fp_line (start -1.6 -1.4) (end -1.6 1.4) (layer F.Fab) (width 0.1))
+    (fp_line (start -1.6 1.4) (end 1.6 1.4) (layer F.Fab) (width 0.1))
+    (fp_line (start 1.6 1.4) (end 1.6 -1.4) (layer F.Fab) (width 0.1))
+    (fp_line (start 1.6 -1.4) (end -1.6 -1.4) (layer F.Fab) (width 0.1))
+    (fp_line (start -1.95 -0.7) (end -1.95 -1.5) (layer F.SilkS) (width 0.12))
+    (fp_line (start -1.95 -1.5) (end 1.95 -1.5) (layer F.SilkS) (width 0.12))
+    (fp_line (start -1.95 1.5) (end 1.95 1.5) (layer F.SilkS) (width 0.12))
+    (fp_text user %R (at 0 0) (layer F.Fab)
+      (effects (font (size 0.5 0.5) (thickness 0.075)))
+    )
+    (pad 1 smd rect (at -1.25 -0.7) (size 1 0.8) (layers F.Cu F.Paste F.Mask)
+      (net 2 "Net-(Pin0-Pad1)"))
+    (pad 4 smd rect (at 1.25 -0.7) (size 1 0.8) (layers F.Cu F.Paste F.Mask)
+      (net 1 +3V3))
+    (pad 3 smd rect (at 1.25 0.7) (size 1 0.8) (layers F.Cu F.Paste F.Mask)
+      (net 4 "Net-(Pin2-Pad1)"))
+    (pad 2 smd rect (at -1.25 0.7) (size 1 0.8) (layers F.Cu F.Paste F.Mask)
+      (net 3 "Net-(Pin1-Pad1)"))
+    (model ${KISYS3DMOD}/LED_SMD.3dshapes/LED_Cree-PLCC4_3.2x2.8mm_CCW.wrl
+      (at (xyz 0 0 0))
+      (scale (xyz 1 1 1))
+      (rotate (xyz 0 0 0))
+    )
   )
   (module TestPoint:TestPoint_Pad_D1.5mm (layer B.Cu)
@@
       (effects (font (size 1 1) (thickness 0.15)) (justify mirror))
     )
+    (fp_circle (center 0 0) (end 1.25 0) (layer B.CrtYd) (width 0.05))
     (fp_circle (center 0 0) (end 0 -0.95) (layer B.SilkS) (width 0.12))
-    (fp_circle (center 0 0) (end 1.25 0) (layer B.CrtYd) (width 0.05))
     (fp_text user %R (at 0 1.65) (layer B.Fab)
       (effects (font (size 1 1) (thickness 0.15)) (justify mirror))
     )
     (pad 1 smd circle (at 0 0) (size 1.5 1.5) (layers B.Cu B.Mask)
-      (net 2 "Net-(Pin1-Pad1)"))
+      (net 3 "Net-(Pin1-Pad1)"))
   )
   (module TestPoint:TestPoint_Pad_D1.5mm (layer B.Cu)
@@
       (effects (font (size 1 1) (thickness 0.15)) (justify mirror))
     )
+    (fp_circle (center 0 0) (end 0 -0.95) (layer B.SilkS) (width 0.12))
     (fp_circle (center 0 0) (end 1.25 0) (layer B.CrtYd) (width 0.05))
-    (fp_circle (center 0 0) (end 0 -0.95) (layer B.SilkS) (width 0.12))
     (fp_text user %R (at 0 1.65) (layer B.Fab)
       (effects (font (size 1 1) (thickness 0.15)) (justify mirror))
     )
     (pad 1 smd circle (at 0 0) (size 1.5 1.5) (layers B.Cu B.Mask)
-      (net 3 "Net-(Pin2-Pad1)"))
+      (net 4 "Net-(Pin2-Pad1)"))
   )
   (gr_text pin2 (at 3.175 -0.508) (layer B.SilkS)
@@
     (effects (font (size 1 1) (thickness 0.15)) (justify right mirror))
   )
-  (segment (start -2.094 -0.7) (end -2.286 -0.508) (width 0.635) (layer F.Cu) (net 1))
-  (segment (start -1.25 -0.7) (end -2.094 -0.7) (width 0.635) (layer F.Cu) (net 1))
-  (via (at -2.286 -0.508) (size 0.6858) (drill 0.3048) (layers F.Cu B.Cu) (net 1))
-  (segment (start -3.048 -1.27) (end -2.286 -0.508) (width 0.635) (layer B.Cu) (net 1))
-  (segment (start -3.175 -1.27) (end -3.048 -1.27) (width 0.635) (layer B.Cu) (net 1))
-  (via (at -2.286 0.381) (size 0.6858) (drill 0.3048) (layers F.Cu B.Cu) (net 2))
-  (segment (start -2.286 0.381) (end -3.175 1.27) (width 0.635) (layer B.Cu) (net 2))
-  (segment (start -1.967 0.7) (end -2.286 0.381) (width 0.635) (layer F.Cu) (net 2))
-  (segment (start -1.25 0.7) (end -1.967 0.7) (width 0.635) (layer F.Cu) (net 2))
-  (via (at 2.286 0.381) (size 0.6858) (drill 0.3048) (layers F.Cu B.Cu) (net 3))
-  (segment (start 1.967 0.7) (end 2.286 0.381) (width 0.635) (layer F.Cu) (net 3))
-  (segment (start 1.25 0.7) (end 1.967 0.7) (width 0.635) (layer F.Cu) (net 3))
-  (segment (start 2.286 0.381) (end 3.175 1.27) (width 0.635) (layer B.Cu) (net 3))
+  (segment (start -2.094 -0.7) (end -2.286 -0.508) (width 0.635) (layer F.Cu) (net 2))
+  (segment (start -1.25 -0.7) (end -2.094 -0.7) (width 0.635) (layer F.Cu) (net 2))
+  (via (at -2.286 -0.508) (size 0.6858) (drill 0.3048) (layers F.Cu B.Cu) (net 2))
+  (segment (start -3.048 -1.27) (end -2.286 -0.508) (width 0.635) (layer B.Cu) (net 2))
+  (segment (start -3.175 -1.27) (end -3.048 -1.27) (width 0.635) (layer B.Cu) (net 2))
+  (via (at -2.286 0.381) (size 0.6858) (drill 0.3048) (layers F.Cu B.Cu) (net 3))
+  (segment (start -2.286 0.381) (end -3.175 1.27) (width 0.635) (layer B.Cu) (net 3))
+  (segment (start -1.967 0.7) (end -2.286 0.381) (width 0.635) (layer F.Cu) (net 3))
+  (segment (start -1.25 0.7) (end -1.967 0.7) (width 0.635) (layer F.Cu) (net 3))
+  (via (at 2.286 0.381) (size 0.6858) (drill 0.3048) (layers F.Cu B.Cu) (net 4))
+  (segment (start 1.967 0.7) (end 2.286 0.381) (width 0.635) (layer F.Cu) (net 4))
+  (segment (start 1.25 0.7) (end 1.967 0.7) (width 0.635) (layer F.Cu) (net 4))
+  (segment (start 2.286 0.381) (end 3.175 1.27) (width 0.635) (layer B.Cu) (net 4))
 )
