File: build-system/erbui/generators/front_pcb/thonk.pj398sm/thonk.pj398sm.wire.kicad_pcb (KiCad board)
At the start: 2 copper layers, 2 parts

Commit message: Update pcbs
Parts:
- added Cascade0: TestPoint, TestPoint:TestPoint_Pad_D1.5mm, B.Cu at (-1.90, 1.80)
- added ZZ2: TestPoint, TestPoint:TestPoint_Pad_D1.5mm, B.Cu at (1.90, 1.80)
Routing:
- net Net-(Pin0-Pad1): track 1.92 -> 7.51 mm
- net Net-(Cascade0-Pad1): track 0.00 -> 2.61 mm
Other:
- board text added: "cascade_from"
- board text added: "cascade_to"
Changed lines of the file:
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@@
   (general
     (thickness 1.6)
-    (drawings 1)
-    (tracks 1)
+    (drawings 3)
+    (tracks 6)
     (zones 0)
-    (modules 2)
+    (modules 4)
     (nets 4)
   )
@@
       (net 2 "Net-(Pin0-Pad1)"))
   )
+  (module TestPoint:TestPoint_Pad_D1.5mm (layer B.Cu)
+    (at -1.9 1.8)
+    (descr "SMD pad as test Point, diameter 1.5mm")
+    (tags "test point SMD pad")
+    (attr virtual)
+    (fp_text reference Cascade0 (at 0 1.648) (layer B.SilkS) hide
+      (effects (font (size 1 1) (thickness 0.15)) (justify mirror))
+    )
+    (fp_text value TestPoint (at 0 -1.75) (layer B.Fab)
+      (effects (font (size 1 1) (thickness 0.15)) (justify mirror))
+    )
+    (fp_circle (center 0 0) (end 1.25 0) (layer B.CrtYd) (width 0.05))
+    (fp_circle (center 0 0) (end 0 -0.95) (layer B.SilkS) (width 0.12))
+    (fp_text user %R (at 0 1.65) (layer B.Fab)
+      (effects (font (size 1 1) (thickness 0.15)) (justify mirror))
+    )
+    (pad 1 smd circle (at 0 0) (size 1.5 1.5) (layers B.Cu B.Mask)
+      (net 3 "Net-(Cascade0-Pad1)"))
+  )
+  (module TestPoint:TestPoint_Pad_D1.5mm (layer B.Cu)
+    (at 1.9 1.8)
+    (descr "SMD pad as test Point, diameter 1.5mm")
+    (tags "test point SMD pad")
+    (attr virtual)
+    (fp_text reference ZZ2 (at 0 1.648) (layer B.SilkS) hide
+      (effects (font (size 1 1) (thickness 0.15)) (justify mirror))
+    )
+    (fp_text value TestPoint (at 0 -1.75) (layer B.Fab)
+      (effects (font (size 1 1) (thickness 0.15)) (justify mirror))
+    )
+    (fp_circle (center 0 0) (end 0 -0.95) (layer B.SilkS) (width 0.12))
+    (fp_circle (center 0 0) (end 1.25 0) (layer B.CrtYd) (width 0.05))
+    (fp_text user %R (at 0 1.65) (layer B.Fab)
+      (effects (font (size 1 1) (thickness 0.15)) (justify mirror))
+    )
+    (pad 1 smd circle (at 0 0) (size 1.5 1.5) (layers B.Cu B.Mask)
+      (net 2 "Net-(Pin0-Pad1)"))
+  )
+  (gr_text cascade_to (at 1.4 0.1) (layer B.SilkS)
+    (effects (font (size 1 1) (thickness 0.15)) (justify right mirror))
+  )
+  (gr_text cascade_from (at -1.4 0.1) (layer B.SilkS)
+    (effects (font (size 1 1) (thickness 0.15)) (justify left mirror))
+  )
   (gr_text pin (at -0.95 -3) (layer B.SilkS)
     (effects (font (size 1 1) (thickness 0.15)) (justify left mirror))
   )
   (segment (start 0 -4.92) (end 0 -3) (width 0.635) (layer B.Cu) (net 2))
+  (segment (start 1.9 -1.1) (end 1.9 1.8) (width 0.635) (layer B.Cu) (net 2))
+  (segment (start 0 -3) (end 1.9 -1.1) (width 0.635) (layer B.Cu) (net 2))
+  (segment (start -0.42 3.38) (end 0 3.38) (width 0.635) (layer B.Cu) (net 3))
+  (segment (start -1.9 1.9) (end -0.42 3.38) (width 0.635) (layer B.Cu) (net 3))
+  (segment (start -1.9 1.8) (end -1.9 1.9) (width 0.635) (layer B.Cu) (net 3))
 )
