File: build-system/erbui/generators/front_pcb/alpha.9mm.manual/alpha.9mm.manual.kicad_pcb (KiCad board)
At the start: 2 copper layers, 1 part

Commit message: Upgrade default manufacturer parts to kicad 6
Other:
- net class Default removed
Changed lines of the file:
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@@
-(kicad_pcb (version 20171130) (host pcbnew "(5.1.9-0-10_14)")
+(kicad_pcb (version 20211014) (generator pcbnew)
   (general
     (thickness 1.6)
-    (drawings 1)
-    (tracks 0)
-    (zones 0)
-    (modules 1)
-    (nets 4)
   )
-  (page A4)
+  (paper "A4")
   (layers
-    (0 F.Cu signal)
-    (31 B.Cu signal)
-    (32 B.Adhes user)
-    (33 F.Adhes user)
-    (34 B.Paste user)
-    (35 F.Paste user)
-    (36 B.SilkS user)
-    (37 F.SilkS user)
-    (38 B.Mask user)
-    (39 F.Mask user)
-    (40 Dwgs.User user)
-    (41 Cmts.User user)
-    (42 Eco1.User user)
-    (43 Eco2.User user)
-    (44 Edge.Cuts user)
-    (45 Margin user)
-    (46 B.CrtYd user hide)
-    (47 F.CrtYd user hide)
-    (48 B.Fab user hide)
-    (49 F.Fab user hide)
+    (0 "F.Cu" signal)
+    (31 "B.Cu" signal)
+    (32 "B.Adhes" user "B.Adhesive")
+    (33 "F.Adhes" user "F.Adhesive")
+    (34 "B.Paste" user)
+    (35 "F.Paste" user)
+    (36 "B.SilkS" user "B.Silkscreen")
+    (37 "F.SilkS" user "F.Silkscreen")
+    (38 "B.Mask" user)
+    (39 "F.Mask" user)
+    (40 "Dwgs.User" user "User.Drawings")
+    (41 "Cmts.User" user "User.Comments")
+    (42 "Eco1.User" user "User.Eco1")
+    (43 "Eco2.User" user "User.Eco2")
+    (44 "Edge.Cuts" user)
+    (45 "Margin" user)
+    (46 "B.CrtYd" user "B.Courtyard")
+    (47 "F.CrtYd" user "F.Courtyard")
+    (48 "B.Fab" user)
+    (49 "F.Fab" user)
   )
   (setup
-    (last_trace_width 0.1524)
-    (user_trace_width 0.1524)
-    (user_trace_width 0.254)
-    (user_trace_width 0.4064)
-    (user_trace_width 0.635)
-    (trace_clearance 0.1524)
-    (zone_clearance 0.508)
-    (zone_45_only no)
-    (trace_min 0.1524)
-    (via_size 0.6858)
-    (via_drill 0.3048)
-    (via_min_size 0.6858)
-    (via_min_drill 0.3048)
-    (uvia_size 0.3048)
-    (uvia_drill 0.1524)
-    (uvias_allowed no)
-    (uvia_min_size 0.2)
-    (uvia_min_drill 0.1)
-    (edge_width 0.15)
-    (segment_width 0.2)
-    (pcb_text_width 0.3)
-    (pcb_text_size 1.5 1.5)
-    (mod_edge_width 0.15)
-    (mod_text_size 1 1)
-    (mod_text_width 0.15)
-    (pad_size 1.7 1.7)
-    (pad_drill 1)
     (pad_to_mask_clearance 0.2)
-    (aux_axis_origin 0 0)
-    (visible_elements FFFFFF7F)
     (pcbplotparams
-      (layerselection 0x010fc_ffffffff)
+      (layerselection 0x00010fc_ffffffff)
+      (disableapertmacros false)
       (usegerberextensions false)
       (usegerberattributes false)
       (usegerberadvancedattributes false)
       (creategerberjobfile false)
+      (svguseinch false)
+      (svgprecision 6)
       (excludeedgelayer true)
-      (linewidth 0.100000)
       (plotframeref false)
       (viasonmask false)
@@
       (hpglpenspeed 20)
       (hpglpendiameter 15.000000)
+      (dxfpolygonmode true)
+      (dxfimperialunits true)
+      (dxfusepcbnewfont true)
       (psnegative false)
       (psa4output false)
@@
       (plotvalue true)
       (plotinvisibletext false)
-      (padsonsilk false)
+      (sketchpadsonfab false)
       (subtractmaskfromsilk false)
       (outputformat 1)
@@
       (drillshape 1)
       (scaleselection 1)
-      (outputdirectory ""))
+      (outputdirectory "")
+    )
   )
   (net 0 "")
-  (net 1 +3V3)
-  (net 2 GND)
-  (net 3 Pin0)
-  (net_class Default "This is the default net class."
-    (clearance 0.1524)
-    (trace_width 0.1524)
-    (via_dia 0.6858)
-    (via_drill 0.3048)
-    (uvia_dia 0.3048)
-    (uvia_drill 0.1524)
-    (diff_pair_width 0.1524)
-    (diff_pair_gap 0.1524)
-    (add_net +3V3)
-    (add_net GND)
-    (add_net Pin0)
-  )
-  (module Potentiometer_Thonk:AlphaPot9ShaftD locked (layer F.Cu)
+  (net 1 "+3V3")
+  (net 2 "GND")
+  (net 3 "Pin0")
+  (footprint "Potentiometer_Thonk:AlphaPot9ShaftD" locked (layer "F.Cu")
     (at 0 0)
-    (fp_text reference RV1 (at 0 4.7) (layer F.SilkS)
+    (attr through_hole)
+    (fp_text reference "RV1" (at 0 4.7) (layer "F.SilkS")
       (effects (font (size 1 1) (thickness 0.15)))
     )
-    (fp_text value 100k (at 0 10.1) (layer F.Fab)
+    (fp_text value "100k" (at 0 10.1) (layer "F.Fab")
       (effects (font (size 1 1) (thickness 0.15)))
     )
-    (fp_line (start -4.7 -4.8) (end 4.7 -4.8) (layer F.SilkS) (width 0.15))
-    (fp_line (start 4.7 -4.8) (end 4.7 -1.4) (layer F.SilkS) (width 0.15))
-    (fp_line (start -4.7 -4.8) (end -4.7 -1.4) (layer F.SilkS) (width 0.15))
-    (fp_line (start -4.7 6.5) (end -3.7 6.5) (layer F.SilkS) (width 0.15))
-    (fp_line (start -4.7 1.4) (end -4.7 6.5) (layer F.SilkS) (width 0.15))
-    (fp_line (start 4.7 1.4) (end 4.7 6.5) (layer F.SilkS) (width 0.15))
-    (fp_line (start 3.7 6.5) (end 4.7 6.5) (layer F.SilkS) (width 0.15))
-    (fp_circle (center 0 0) (end 3 0) (layer F.SilkS) (width 0.15))
-    (fp_line (start -2.6 1.5) (end 2.6 1.5) (layer F.SilkS) (width 0.15))
-    (fp_circle (center 3.8 -3.8) (end 4.2 -3.8) (layer F.SilkS) (width 0.15))
-    (fp_circle (center -3.8 5.6) (end -4.2 5.6) (layer F.SilkS) (width 0.15))
-    (fp_arc (start 0 0) (end -1.6 1.5) (angle 265) (layer F.SilkS) (width 0.15))
-    (pad "" thru_hole oval (at 5.7 0) (size 2.5 1.8) (drill oval 1.8 1.1) (layers *.Cu *.Mask))
-    (pad 3 thru_hole oval (at 2.5 7.5) (size 1.7 1.7) (drill 1) (layers *.Cu *.Mask)
-      (net 1 +3V3))
-    (pad 2 thru_hole oval (at 0 7.5) (size 1.7 1.7) (drill 1) (layers *.Cu *.Mask)
-      (net 3 Pin0))
-    (pad 1 thru_hole oval (at -2.5 7.5) (size 1.7 1.7) (drill 1) (layers *.Cu *.Mask)
-      (net 2 GND))
-    (pad "" thru_hole oval (at -5.7 0) (size 2.5 1.8) (drill oval 1.8 1.1) (layers *.Cu *.Mask))
+    (fp_line (start -4.7 -4.8) (end 4.7 -4.8) (layer "F.SilkS") (width 0.15))
+    (fp_line (start -4.7 -4.8) (end -4.7 -1.4) (layer "F.SilkS") (width 0.15))
+    (fp_line (start -2.6 1.5) (end 2.6 1.5) (layer "F.SilkS") (width 0.15))
+    (fp_line (start 4.7 1.4) (end 4.7 6.5) (layer "F.SilkS") (width 0.15))
+    (fp_line (start -4.7 1.4) (end -4.7 6.5) (layer "F.SilkS") (width 0.15))
+    (fp_line (start -4.7 6.5) (end -3.7 6.5) (layer "F.SilkS") (width 0.15))
+    (fp_line (start 3.7 6.5) (end 4.7 6.5) (layer "F.SilkS") (width 0.15))
+    (fp_line (start 4.7 -4.8) (end 4.7 -1.4) (layer "F.SilkS") (width 0.15))
+    (fp_arc (start -1.6 1.5) (mid -0.024972 -2.193029) (end 1.633741 1.463178) (layer "F.SilkS") (width 0.15))
+    (fp_circle (center 3.8 -3.8) (end 4.2 -3.8) (layer "F.SilkS") (width 0.15) (fill none))
+    (fp_circle (center -3.8 5.6) (end -4.2 5.6) (layer "F.SilkS") (width 0.15) (fill none))
+    (fp_circle (center 0 0) (end 3 0) (layer "F.SilkS") (width 0.15) (fill none))
+    (pad "" thru_hole oval locked (at -5.7 0) (size 2.5 1.8) (drill oval 1.8 1.1) (layers *.Cu *.Mask))
+    (pad "" thru_hole oval locked (at 5.7 0) (size 2.5 1.8) (drill oval 1.8 1.1) (layers *.Cu *.Mask))
+    (pad "1" thru_hole oval locked (at -2.5 7.5) (size 1.7 1.7) (drill 1) (layers *.Cu *.Mask)
+      (net 2 "GND"))
+    (pad "2" thru_hole oval locked (at 0 7.5) (size 1.7 1.7) (drill 1) (layers *.Cu *.Mask)
+      (net 3 "Pin0"))
+    (pad "3" thru_hole oval locked (at 2.5 7.5) (size 1.7 1.7) (drill 1) (layers *.Cu *.Mask)
+      (net 1 "+3V3"))
   )
-  (gr_circle (center 0 0) (end 3.75 0) (layer Eco1.User) (width 0.12))
+  (gr_circle (center 0 0) (end 3.75 0) (layer "Eco1.User") (width 0.12) (fill none))
 )
