File: build-system/erbui/generators/front_pcb/dailywell.2ms1.wire/dailywell.2ms1.wire.kicad_pcb (KiCad board)
At the start: 2 copper layers, 3 parts, among them SW1 SW_SPDT

Commit message: Wip
Other:
- net class Default removed
