File: build-system/erbui/generators/front_pcb/dailywell.2ms3.manual/dailywell.2ms3.manual.kicad_pcb (KiCad board)
At the start: 2 copper layers, 1 part, among them SW1 SW_SPDT

Commit message: Wip
Other:
- net class Default removed
Changed lines of the file:
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@@
-(kicad_pcb (version 20171130) (host pcbnew "(5.1.9-0-10_14)")
+(kicad_pcb (version 20211014) (generator pcbnew)
   (general
     (thickness 1.6)
-    (drawings 0)
-    (tracks 0)
-    (zones 0)
-    (modules 1)
-    (nets 4)
   )
-  (page A4)
+  (paper "A4")
   (layers
-    (0 F.Cu signal)
-    (31 B.Cu signal)
-    (32 B.Adhes user)
-    (33 F.Adhes user)
-    (34 B.Paste user)
-    (35 F.Paste user)
-    (36 B.SilkS user)
-    (37 F.SilkS user)
-    (38 B.Mask user)
-    (39 F.Mask user)
-    (40 Dwgs.User user)
-    (41 Cmts.User user)
-    (42 Eco1.User user)
-    (43 Eco2.User user)
-    (44 Edge.Cuts user)
-    (45 Margin user)
-    (46 B.CrtYd user hide)
-    (47 F.CrtYd user hide)
-    (48 B.Fab user hide)
-    (49 F.Fab user hide)
+    (0 "F.Cu" signal)
+    (31 "B.Cu" signal)
+    (32 "B.Adhes" user "B.Adhesive")
+    (33 "F.Adhes" user "F.Adhesive")
+    (34 "B.Paste" user)
+    (35 "F.Paste" user)
+    (36 "B.SilkS" user "B.Silkscreen")
+    (37 "F.SilkS" user "F.Silkscreen")
+    (38 "B.Mask" user)
+    (39 "F.Mask" user)
+    (40 "Dwgs.User" user "User.Drawings")
+    (41 "Cmts.User" user "User.Comments")
+    (42 "Eco1.User" user "User.Eco1")
+    (43 "Eco2.User" user "User.Eco2")
+    (44 "Edge.Cuts" user)
+    (45 "Margin" user)
+    (46 "B.CrtYd" user "B.Courtyard")
+    (47 "F.CrtYd" user "F.Courtyard")
+    (48 "B.Fab" user)
+    (49 "F.Fab" user)
   )
   (setup
-    (last_trace_width 0.1524)
-    (user_trace_width 0.1524)
-    (user_trace_width 0.254)
-    (user_trace_width 0.4064)
-    (user_trace_width 0.635)
-    (trace_clearance 0.1524)
-    (zone_clearance 0.508)
-    (zone_45_only no)
-    (trace_min 0.1524)
-    (via_size 0.6858)
-    (via_drill 0.3048)
-    (via_min_size 0.6858)
-    (via_min_drill 0.3048)
-    (uvia_size 0.3048)
-    (uvia_drill 0.1524)
-    (uvias_allowed no)
-    (uvia_min_size 0.2)
-    (uvia_min_drill 0.1)
-    (edge_width 0.15)
-    (segment_width 0.15)
-    (pcb_text_width 0.3)
-    (pcb_text_size 1.5 1.5)
-    (mod_edge_width 0.15)
-    (mod_text_size 1 1)
-    (mod_text_width 0.15)
-    (pad_size 1.524 1.524)
-    (pad_drill 0.762)
     (pad_to_mask_clearance 0.2)
-    (aux_axis_origin 0 0)
-    (visible_elements FFFFFF7F)
     (pcbplotparams
-      (layerselection 0x010fc_ffffffff)
+      (layerselection 0x00010fc_ffffffff)
+      (disableapertmacros false)
       (usegerberextensions false)
       (usegerberattributes false)
       (usegerberadvancedattributes false)
       (creategerberjobfile false)
+      (svguseinch false)
+      (svgprecision 6)
       (excludeedgelayer true)
-      (linewidth 0.100000)
       (plotframeref false)
       (viasonmask false)
@@
       (hpglpenspeed 20)
       (hpglpendiameter 15.000000)
+      (dxfpolygonmode true)
+      (dxfimperialunits true)
+      (dxfusepcbnewfont true)
       (psnegative false)
       (psa4output false)
@@
       (plotvalue true)
       (plotinvisibletext false)
-      (padsonsilk false)
+      (sketchpadsonfab false)
       (subtractmaskfromsilk false)
       (outputformat 1)
@@
       (drillshape 1)
       (scaleselection 1)
-      (outputdirectory ""))
+      (outputdirectory "")
+    )
   )
   (net 0 "")
-  (net 1 +3V3)
-  (net 2 Pin1)
-  (net 3 Pin0)
-  (net_class Default "This is the default net class."
-    (clearance 0.1524)
-    (trace_width 0.1524)
-    (via_dia 0.6858)
-    (via_drill 0.3048)
-    (uvia_dia 0.3048)
-    (uvia_drill 0.1524)
-    (diff_pair_width 0.1524)
-    (diff_pair_gap 0.1524)
-    (add_net +3V3)
-    (add_net Pin0)
-    (add_net Pin1)
-  )
-  (module Switch_Thonk:SW_SPDT_Dailywell locked (layer F.Cu)
+  (net 1 "+3V3")
+  (net 2 "Pin1")
+  (net 3 "Pin0")
+  (footprint "Switch_Thonk:SW_SPDT_Dailywell" locked (layer "F.Cu")
     (at 0 0)
-    (fp_text reference SW1 (at 0 5.08) (layer F.SilkS)
+    (attr through_hole)
+    (fp_text reference "SW1" (at 0 5.08) (layer "F.SilkS")
       (effects (font (size 1 1) (thickness 0.15)))
     )
-    (fp_text value SW_SPDT (at 0 -5.08) (layer F.Fab)
+    (fp_text value "SW_SPDT" (at 0 -5.08) (layer "F.Fab")
       (effects (font (size 1 1) (thickness 0.15)))
     )
-    (fp_line (start -2.0701 -1.35128) (end -2.0701 1.35128) (layer F.SilkS) (width 0.15))
-    (fp_line (start 2.54 -4.064) (end 2.54 4.064) (layer F.SilkS) (width 0.15))
-    (fp_line (start -2.54 -4.064) (end -2.54 4.064) (layer F.SilkS) (width 0.15))
-    (fp_line (start -2.54 4.064) (end 2.54 4.064) (layer F.SilkS) (width 0.15))
-    (fp_line (start -2.54 -4.064) (end 2.54 -4.064) (layer F.SilkS) (width 0.15))
-    (fp_arc (start 0 0) (end 2.4765 0) (angle -65.38985762) (layer F.SilkS) (width 0.15))
-    (fp_arc (start 0 0) (end -1.033779 -2.245359) (angle -32.27419574) (layer F.SilkS) (width 0.15))
-    (fp_arc (start 0 0) (end 2.4765 0) (angle 65.4) (layer F.SilkS) (width 0.15))
-    (fp_arc (start 0 0) (end -2.070099 1.358899) (angle -32.3) (layer F.SilkS) (width 0.15))
-    (fp_line (start -3.5 -4) (end 3.5 -4) (layer Dwgs.User) (width 0.12))
-    (fp_line (start 3.5 -4) (end 3.5 4) (layer Dwgs.User) (width 0.12))
-    (fp_line (start 3.5 4) (end -3.5 4) (layer Dwgs.User) (width 0.12))
-    (fp_line (start -3.5 4) (end -3.5 -4) (layer Dwgs.User) (width 0.12))
-    (pad 2 thru_hole circle (at 0 0) (size 1.8796 1.8796) (drill 1.0922) (layers *.Cu *.Mask)
-      (net 1 +3V3))
-    (pad 3 thru_hole circle (at 0 -2.54) (size 1.8796 1.8796) (drill 1.0922) (layers *.Cu *.Mask)
-      (net 2 Pin1))
-    (pad 1 thru_hole circle (at 0 2.54) (size 1.8796 1.8796) (drill 1.0922) (layers *.Cu *.Mask)
-      (net 3 Pin0))
+    (fp_line (start -2.54 -4.064) (end 2.54 -4.064) (layer "F.SilkS") (width 0.15))
+    (fp_line (start -2.0701 -1.35128) (end -2.0701 1.35128) (layer "F.SilkS") (width 0.15))
+    (fp_line (start -2.54 4.064) (end 2.54 4.064) (layer "F.SilkS") (width 0.15))
+    (fp_line (start -2.54 -4.064) (end -2.54 4.064) (layer "F.SilkS") (width 0.15))
+    (fp_line (start 2.54 -4.064) (end 2.54 4.064) (layer "F.SilkS") (width 0.15))
+    (fp_arc (start -1.023645 2.254788) (mid -1.610425 1.881077) (end -2.070099 1.358899) (layer "F.SilkS") (width 0.15))
+    (fp_arc (start -2.073021 -1.346448) (mid -1.617115 -1.869566) (end -1.033779 -2.245359) (layer "F.SilkS") (width 0.15))
+    (fp_arc (start 2.4765 0) (mid 2.084001 1.337905) (end 1.030919 2.251723) (layer "F.SilkS") (width 0.15))
+    (fp_arc (start 1.031318 -2.251541) (mid 2.08412 -1.337721) (end 2.4765 0) (layer "F.SilkS") (width 0.15))
+    (fp_line (start 3.5 4) (end -3.5 4) (layer "Dwgs.User") (width 0.12))
+    (fp_line (start -3.5 4) (end -3.5 -4) (layer "Dwgs.User") (width 0.12))
+    (fp_line (start 3.5 -4) (end 3.5 4) (layer "Dwgs.User") (width 0.12))
+    (fp_line (start -3.5 -4) (end 3.5 -4) (layer "Dwgs.User") (width 0.12))
+    (pad "1" thru_hole circle locked (at 0 2.54) (size 1.8796 1.8796) (drill 1.0922) (layers *.Cu *.Mask)
+      (net 3 "Pin0"))
+    (pad "2" thru_hole circle locked (at 0 0) (size 1.8796 1.8796) (drill 1.0922) (layers *.Cu *.Mask)
+      (net 1 "+3V3"))
+    (pad "3" thru_hole circle locked (at 0 -2.54) (size 1.8796 1.8796) (drill 1.0922) (layers *.Cu *.Mask)
+      (net 2 "Pin1"))
   )
-  (gr_circle (center 0 0) (end 2.475 0) (layer Eco1.User) (width 0.12))
+  (gr_circle (center 0 0) (end 2.475 0) (layer "Eco1.User") (width 0.12) (fill none))
 )
