File: build-system/erbui/generators/front_pcb/led.3mm.rgb.manual/led.3mm.rgb.manual.kicad_pcb (KiCad board)
At the start: 2 copper layers, 1 part

Commit message: Wip
Other:
- net class Default removed
Changed lines of the file:
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@@
-(kicad_pcb (version 20171130) (host pcbnew "(5.1.9-0-10_14)")
+(kicad_pcb (version 20211014) (generator pcbnew)
   (general
     (thickness 1.6)
-    (drawings 0)
-    (tracks 0)
-    (zones 0)
-    (modules 1)
-    (nets 5)
   )
-  (page A4)
+  (paper "A4")
   (layers
-    (0 F.Cu signal)
-    (31 B.Cu signal)
-    (32 B.Adhes user)
-    (33 F.Adhes user)
-    (34 B.Paste user)
-    (35 F.Paste user)
-    (36 B.SilkS user)
-    (37 F.SilkS user)
-    (38 B.Mask user)
-    (39 F.Mask user)
-    (40 Dwgs.User user)
-    (41 Cmts.User user)
-    (42 Eco1.User user)
-    (43 Eco2.User user)
-    (44 Edge.Cuts user)
-    (45 Margin user)
-    (46 B.CrtYd user hide)
-    (47 F.CrtYd user hide)
-    (48 B.Fab user hide)
-    (49 F.Fab user hide)
+    (0 "F.Cu" signal)
+    (31 "B.Cu" signal)
+    (32 "B.Adhes" user "B.Adhesive")
+    (33 "F.Adhes" user "F.Adhesive")
+    (34 "B.Paste" user)
+    (35 "F.Paste" user)
+    (36 "B.SilkS" user "B.Silkscreen")
+    (37 "F.SilkS" user "F.Silkscreen")
+    (38 "B.Mask" user)
+    (39 "F.Mask" user)
+    (40 "Dwgs.User" user "User.Drawings")
+    (41 "Cmts.User" user "User.Comments")
+    (42 "Eco1.User" user "User.Eco1")
+    (43 "Eco2.User" user "User.Eco2")
+    (44 "Edge.Cuts" user)
+    (45 "Margin" user)
+    (46 "B.CrtYd" user "B.Courtyard")
+    (47 "F.CrtYd" user "F.Courtyard")
+    (48 "B.Fab" user)
+    (49 "F.Fab" user)
   )
   (setup
-    (last_trace_width 0.1524)
-    (user_trace_width 0.1524)
-    (user_trace_width 0.254)
-    (user_trace_width 0.4064)
-    (user_trace_width 0.635)
-    (trace_clearance 0.1524)
-    (zone_clearance 0.508)
-    (zone_45_only no)
-    (trace_min 0.1524)
-    (via_size 0.6858)
-    (via_drill 0.3048)
-    (via_min_size 0.6858)
-    (via_min_drill 0.3048)
-    (uvia_size 0.3048)
-    (uvia_drill 0.1524)
-    (uvias_allowed no)
-    (uvia_min_size 0.2)
-    (uvia_min_drill 0.1)
-    (edge_width 0.15)
-    (segment_width 0.15)
-    (pcb_text_width 0.3)
-    (pcb_text_size 1.5 1.5)
-    (mod_edge_width 0.15)
-    (mod_text_size 1 1)
-    (mod_text_width 0.15)
-    (pad_size 1.8 1.8)
-    (pad_drill 0.9)
     (pad_to_mask_clearance 0.2)
-    (aux_axis_origin 0 0)
-    (visible_elements FFFFFF7F)
     (pcbplotparams
-      (layerselection 0x010fc_ffffffff)
+      (layerselection 0x00010fc_ffffffff)
+      (disableapertmacros false)
       (usegerberextensions false)
       (usegerberattributes false)
       (usegerberadvancedattributes false)
       (creategerberjobfile false)
+      (svguseinch false)
+      (svgprecision 6)
       (excludeedgelayer true)
-      (linewidth 0.100000)
       (plotframeref false)
       (viasonmask false)
@@
       (hpglpenspeed 20)
       (hpglpendiameter 15.000000)
+      (dxfpolygonmode true)
+      (dxfimperialunits true)
+      (dxfusepcbnewfont true)
       (psnegative false)
       (psa4output false)
@@
       (plotvalue true)
       (plotinvisibletext false)
-      (padsonsilk false)
+      (sketchpadsonfab false)
       (subtractmaskfromsilk false)
       (outputformat 1)
@@
       (drillshape 1)
       (scaleselection 1)
-      (outputdirectory ""))
+      (outputdirectory "")
+    )
   )
   (net 0 "")
-  (net 1 +3V3)
-  (net 2 Pin0)
-  (net 3 Pin2)
-  (net 4 Pin1)
-  (net_class Default "This is the default net class."
-    (clearance 0.1524)
-    (trace_width 0.1524)
-    (via_dia 0.6858)
-    (via_drill 0.3048)
-    (uvia_dia 0.3048)
-    (uvia_drill 0.1524)
-    (diff_pair_width 0.1524)
-    (diff_pair_gap 0.1524)
-    (add_net +3V3)
-    (add_net Pin0)
-    (add_net Pin1)
-    (add_net Pin2)
-  )
-  (module LED_SMD:LED_Cree-PLCC4_3.2x2.8mm_CCW locked (layer F.Cu)
+  (net 1 "+3V3")
+  (net 2 "Pin0")
+  (net 3 "Pin2")
+  (net 4 "Pin1")
+  (footprint "LED_SMD:LED_Cree-PLCC4_3.2x2.8mm_CCW" locked (layer "F.Cu")
     (at 0 0)
     (descr "3.2mm x 2.8mm PLCC4 LED, http://www.cree.com/led-components/media/documents/CLV1AFKB(874).pdf")
     (tags "LED Cree PLCC-4")
     (attr smd)
-    (fp_text reference D1 (at 0 -2.65) (layer F.SilkS)
+    (fp_text reference "D1" (at 0 -2.65) (layer "F.SilkS")
       (effects (font (size 1 1) (thickness 0.15)))
     )
-    (fp_text value LED_RGBA (at 0 2.65) (layer F.Fab)
+    (fp_text value "LED_RGBA" (at 0 2.65) (layer "F.Fab")
       (effects (font (size 1 1) (thickness 0.15)))
     )
-    (fp_line (start -1.95 1.5) (end 1.95 1.5) (layer F.SilkS) (width 0.12))
-    (fp_line (start -1.95 -1.5) (end 1.95 -1.5) (layer F.SilkS) (width 0.12))
-    (fp_line (start -1.95 -0.7) (end -1.95 -1.5) (layer F.SilkS) (width 0.12))
-    (fp_line (start 1.6 -1.4) (end -1.6 -1.4) (layer F.Fab) (width 0.1))
-    (fp_line (start 1.6 1.4) (end 1.6 -1.4) (layer F.Fab) (width 0.1))
-    (fp_line (start -1.6 1.4) (end 1.6 1.4) (layer F.Fab) (width 0.1))
-    (fp_line (start -1.6 -1.4) (end -1.6 1.4) (layer F.Fab) (width 0.1))
-    (fp_line (start -0.6 -1.4) (end -1.6 -0.4) (layer F.Fab) (width 0.1))
-    (fp_line (start 2.2 -1.75) (end -2.2 -1.75) (layer F.CrtYd) (width 0.05))
-    (fp_line (start 2.2 1.75) (end 2.2 -1.75) (layer F.CrtYd) (width 0.05))
-    (fp_line (start -2.2 1.75) (end 2.2 1.75) (layer F.CrtYd) (width 0.05))
-    (fp_line (start -2.2 -1.75) (end -2.2 1.75) (layer F.CrtYd) (width 0.05))
-    (fp_circle (center 0 0) (end 1.12 0) (layer F.Fab) (width 0.1))
-    (fp_text user %R (at 0 0) (layer F.Fab)
+    (fp_text user "${REFERENCE}" (at 0 0) (layer "F.Fab")
       (effects (font (size 0.5 0.5) (thickness 0.075)))
     )
-    (fp_circle (center 0 0) (end 1.5 0) (layer Dwgs.User) (width 0.15))
-    (pad 1 smd rect (at -1.25 -0.7) (size 1 0.8) (layers F.Cu F.Paste F.Mask)
-      (net 2 Pin0))
-    (pad 4 smd rect (at 1.25 -0.7) (size 1 0.8) (layers F.Cu F.Paste F.Mask)
-      (net 1 +3V3))
-    (pad 3 smd rect (at 1.25 0.7) (size 1 0.8) (layers F.Cu F.Paste F.Mask)
-      (net 3 Pin2))
-    (pad 2 smd rect (at -1.25 0.7) (size 1 0.8) (layers F.Cu F.Paste F.Mask)
-      (net 4 Pin1))
-    (model ${KISYS3DMOD}/LED_SMD.3dshapes/LED_Cree-PLCC4_3.2x2.8mm_CCW.wrl
-      (at (xyz 0 0 0))
+    (fp_line (start -1.95 1.5) (end 1.95 1.5) (layer "F.SilkS") (width 0.12))
+    (fp_line (start -1.95 -1.5) (end 1.95 -1.5) (layer "F.SilkS") (width 0.12))
+    (fp_line (start -1.95 -0.7) (end -1.95 -1.5) (layer "F.SilkS") (width 0.12))
+    (fp_circle (center 0 0) (end 1.5 0) (layer "Dwgs.User") (width 0.15) (fill none))
+    (fp_line (start 2.2 -1.75) (end -2.2 -1.75) (layer "F.CrtYd") (width 0.05))
+    (fp_line (start -2.2 -1.75) (end -2.2 1.75) (layer "F.CrtYd") (width 0.05))
+    (fp_line (start 2.2 1.75) (end 2.2 -1.75) (layer "F.CrtYd") (width 0.05))
+    (fp_line (start -2.2 1.75) (end 2.2 1.75) (layer "F.CrtYd") (width 0.05))
+    (fp_line (start 1.6 1.4) (end 1.6 -1.4) (layer "F.Fab") (width 0.1))
+    (fp_line (start -1.6 -1.4) (end -1.6 1.4) (layer "F.Fab") (width 0.1))
+    (fp_line (start -0.6 -1.4) (end -1.6 -0.4) (layer "F.Fab") (width 0.1))
+    (fp_line (start -1.6 1.4) (end 1.6 1.4) (layer "F.Fab") (width 0.1))
+    (fp_line (start 1.6 -1.4) (end -1.6 -1.4) (layer "F.Fab") (width 0.1))
+    (fp_circle (center 0 0) (end 1.12 0) (layer "F.Fab") (width 0.1) (fill none))
+    (pad "1" smd rect locked (at -1.25 -0.7) (size 1 0.8) (layers "F.Cu" "F.Paste" "F.Mask")
+      (net 2 "Pin0"))
+    (pad "2" smd rect locked (at -1.25 0.7) (size 1 0.8) (layers "F.Cu" "F.Paste" "F.Mask")
+      (net 4 "Pin1"))
+    (pad "3" smd rect locked (at 1.25 0.7) (size 1 0.8) (layers "F.Cu" "F.Paste" "F.Mask")
+      (net 3 "Pin2"))
+    (pad "4" smd rect locked (at 1.25 -0.7) (size 1 0.8) (layers "F.Cu" "F.Paste" "F.Mask")
+      (net 1 "+3V3"))
+    (model "${KISYS3DMOD}/LED_SMD.3dshapes/LED_Cree-PLCC4_3.2x2.8mm_CCW.wrl"
+      (offset (xyz 0 0 0))
       (scale (xyz 1 1 1))
       (rotate (xyz 0 0 0))
     )
   )
-  (gr_circle (center 0 0) (end 1.55 0) (layer Eco1.User) (width 0.12))
+  (gr_circle (center 0 0) (end 1.55 0) (layer "Eco1.User") (width 0.12) (fill none))
 )
