File: build-system/erbui/generators/front_pcb/led.3mm.rgb.manual/led.3mm.rgb.manual.kicad_sch (KiCad schematic)
At the start: 1 part

Commit message: Remove deprecated simulator class field from schematic files
Parts:
- D1: Simulator erb::Led3mm <RedGreenBlueLight> -> (none)
Changed lines of the file:
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@@
-      (effects (font (size 1.27 1.27)) hide)
-    )
-    (property "Simulator" "erb::Led3mm <RedGreenBlueLight>" (id 4) (at 157.48 119.38 0)
       (effects (font (size 1.27 1.27)) hide)
     )
