File: build-system/erbui/generators/front_pcb/led.3mm.orange.wire/led.3mm.orange.wire.kicad_pcb (KiCad board)
At the start: 2 copper layers, 2 parts

Commit message: Update erbui front pcb generator parts to kicad 6
Other:
- net class Default removed
Changed lines of the file:
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@@
-(kicad_pcb (version 20171130) (host pcbnew "(5.1.9-0-10_14)")
+(kicad_pcb (version 20211014) (generator pcbnew)
   (general
     (thickness 1.6)
-    (drawings 1)
-    (tracks 1)
-    (zones 0)
-    (modules 2)
-    (nets 3)
   )
-  (page A4)
+  (paper "A4")
   (layers
-    (0 F.Cu signal)
-    (31 B.Cu signal)
-    (32 B.Adhes user)
-    (33 F.Adhes user)
-    (34 B.Paste user)
-    (35 F.Paste user)
-    (36 B.SilkS user)
-    (37 F.SilkS user)
-    (38 B.Mask user)
-    (39 F.Mask user)
-    (40 Dwgs.User user)
-    (41 Cmts.User user)
-    (42 Eco1.User user)
-    (43 Eco2.User user)
-    (44 Edge.Cuts user)
-    (45 Margin user)
-    (46 B.CrtYd user hide)
-    (47 F.CrtYd user hide)
-    (48 B.Fab user hide)
-    (49 F.Fab user hide)
+    (0 "F.Cu" signal)
+    (31 "B.Cu" signal)
+    (32 "B.Adhes" user "B.Adhesive")
+    (33 "F.Adhes" user "F.Adhesive")
+    (34 "B.Paste" user)
+    (35 "F.Paste" user)
+    (36 "B.SilkS" user "B.Silkscreen")
+    (37 "F.SilkS" user "F.Silkscreen")
+    (38 "B.Mask" user)
+    (39 "F.Mask" user)
+    (40 "Dwgs.User" user "User.Drawings")
+    (41 "Cmts.User" user "User.Comments")
+    (42 "Eco1.User" user "User.Eco1")
+    (43 "Eco2.User" user "User.Eco2")
+    (44 "Edge.Cuts" user)
+    (45 "Margin" user)
+    (46 "B.CrtYd" user "B.Courtyard")
+    (47 "F.CrtYd" user "F.Courtyard")
+    (48 "B.Fab" user)
+    (49 "F.Fab" user)
   )
   (setup
-    (last_trace_width 0.1524)
-    (user_trace_width 0.1524)
-    (user_trace_width 0.254)
-    (user_trace_width 0.4064)
-    (user_trace_width 0.635)
-    (trace_clearance 0.1524)
-    (zone_clearance 0.508)
-    (zone_45_only no)
-    (trace_min 0.1524)
-    (via_size 0.6858)
-    (via_drill 0.3048)
-    (via_min_size 0.6858)
-    (via_min_drill 0.3048)
-    (uvia_size 0.3048)
-    (uvia_drill 0.1524)
-    (uvias_allowed no)
-    (uvia_min_size 0.2)
-    (uvia_min_drill 0.1)
-    (edge_width 0.15)
-    (segment_width 0.15)
-    (pcb_text_width 0.3)
-    (pcb_text_size 1.5 1.5)
-    (mod_edge_width 0.15)
-    (mod_text_size 1 1)
-    (mod_text_width 0.15)
-    (pad_size 1.524 1.524)
-    (pad_drill 0.762)
     (pad_to_mask_clearance 0.2)
-    (aux_axis_origin 0 0)
-    (visible_elements FFFFFF7F)
     (pcbplotparams
-      (layerselection 0x010fc_ffffffff)
+      (layerselection 0x00010fc_ffffffff)
+      (disableapertmacros false)
       (usegerberextensions false)
       (usegerberattributes false)
       (usegerberadvancedattributes false)
       (creategerberjobfile false)
+      (svguseinch false)
+      (svgprecision 6)
       (excludeedgelayer true)
-      (linewidth 0.100000)
       (plotframeref false)
       (viasonmask false)
@@
       (hpglpenspeed 20)
       (hpglpendiameter 15.000000)
+      (dxfpolygonmode true)
+      (dxfimperialunits true)
+      (dxfusepcbnewfont true)
       (psnegative false)
       (psa4output false)
@@
       (plotvalue true)
       (plotinvisibletext false)
-      (padsonsilk false)
+      (sketchpadsonfab false)
       (subtractmaskfromsilk false)
       (outputformat 1)
@@
       (drillshape 1)
       (scaleselection 1)
-      (outputdirectory ""))
+      (outputdirectory "")
+    )
   )
   (net 0 "")
-  (net 1 GND)
-  (net 2 Pin0)
-  (net_class Default "This is the default net class."
-    (clearance 0.1524)
-    (trace_width 0.1524)
-    (via_dia 0.6858)
-    (via_drill 0.3048)
-    (uvia_dia 0.3048)
-    (uvia_drill 0.1524)
-    (diff_pair_width 0.1524)
-    (diff_pair_gap 0.1524)
-    (add_net GND)
-    (add_net Pin0)
-  )
-  (module LED_THT:LED_D3.0mm locked (layer F.Cu)
+  (net 1 "GND")
+  (net 2 "Pin0")
+  (footprint "LED_THT:LED_D3.0mm" locked (layer "F.Cu")
     (at -1.27 0)
     (descr "LED, diameter 3.0mm, 2 pins")
     (tags "LED diameter 3.0mm 2 pins")
-    (fp_text reference D1 (at 1.27 -2.96) (layer F.SilkS)
+    (attr through_hole)
+    (fp_text reference "D1" (at 1.27 -2.96) (layer "F.SilkS")
       (effects (font (size 1 1) (thickness 0.15)))
     )
-    (fp_text value LED (at 1.27 2.96) (layer F.Fab)
+    (fp_text value "LED" (at 1.27 2.96) (layer "F.Fab")
       (effects (font (size 1 1) (thickness 0.15)))
     )
-    (fp_line (start 3.7 -2.25) (end -1.15 -2.25) (layer F.CrtYd) (width 0.05))
-    (fp_line (start 3.7 2.25) (end 3.7 -2.25) (layer F.CrtYd) (width 0.05))
-    (fp_line (start -1.15 2.25) (end 3.7 2.25) (layer F.CrtYd) (width 0.05))
-    (fp_line (start -1.15 -2.25) (end -1.15 2.25) (layer F.CrtYd) (width 0.05))
-    (fp_line (start -0.29 1.08) (end -0.29 1.236) (layer F.SilkS) (width 0.12))
-    (fp_line (start -0.29 -1.236) (end -0.29 -1.08) (layer F.SilkS) (width 0.12))
-    (fp_line (start -0.23 -1.16619) (end -0.23 1.16619) (layer F.Fab) (width 0.1))
-    (fp_circle (center 1.27 0) (end 2.77 0) (layer F.Fab) (width 0.1))
-    (fp_arc (start 1.27 0) (end -0.23 -1.16619) (angle 284.3) (layer F.Fab) (width 0.1))
-    (fp_arc (start 1.27 0) (end -0.29 -1.235516) (angle 108.8) (layer F.SilkS) (width 0.12))
-    (fp_arc (start 1.27 0) (end -0.29 1.235516) (angle -108.8) (layer F.SilkS) (width 0.12))
-    (fp_arc (start 1.27 0) (end 0.229039 -1.08) (angle 87.9) (layer F.SilkS) (width 0.12))
-    (fp_arc (start 1.27 0) (end 0.229039 1.08) (angle -87.9) (layer F.SilkS) (width 0.12))
-    (fp_circle (center 0 0) (end 1.5 0) (layer Dwgs.User) (width 0.15))
-    (pad 1 thru_hole rect (at 0 0) (size 1.8 1.8) (drill 0.9) (layers *.Cu *.Mask)
-      (net 1 GND))
-    (pad 2 thru_hole circle (at 2.54 0) (size 1.8 1.8) (drill 0.9) (layers *.Cu *.Mask)
-      (net 2 Pin0))
-    (model ${KISYS3DMOD}/LED_THT.3dshapes/LED_D3.0mm.wrl
-      (at (xyz 0 0 0))
+    (fp_line (start -0.29 1.08) (end -0.29 1.236) (layer "F.SilkS") (width 0.12))
+    (fp_line (start -0.29 -1.236) (end -0.29 -1.08) (layer "F.SilkS") (width 0.12))
+    (fp_arc (start 2.31113 1.079837) (mid 1.270117 1.5) (end 0.229039 1.08) (layer "F.SilkS") (width 0.12))
+    (fp_arc (start -0.29 -1.235516) (mid 1.366487 -1.987659) (end 2.942335 -1.078608) (layer "F.SilkS") (width 0.12))
+    (fp_arc (start 0.229039 -1.08) (mid 1.270117 -1.5) (end 2.31113 -1.079837) (layer "F.SilkS") (width 0.12))
+    (fp_arc (start 2.942335 1.078608) (mid 1.366487 1.987659) (end -0.29 1.235516) (layer "F.SilkS") (width 0.12))
+    (fp_circle (center 1.27 0) (end 2.77 0) (layer "Dwgs.User") (width 0.12) (fill none))
+    (fp_line (start -1.15 -2.25) (end -1.15 2.25) (layer "F.CrtYd") (width 0.05))
+    (fp_line (start 3.7 2.25) (end 3.7 -2.25) (layer "F.CrtYd") (width 0.05))
+    (fp_line (start -1.15 2.25) (end 3.7 2.25) (layer "F.CrtYd") (width 0.05))
+    (fp_line (start 3.7 -2.25) (end -1.15 -2.25) (layer "F.CrtYd") (width 0.05))
+    (fp_line (start -0.23 -1.16619) (end -0.23 1.16619) (layer "F.Fab") (width 0.1))
+    (fp_arc (start -0.23 -1.16619) (mid 3.17 0.000452) (end -0.230555 1.165476) (layer "F.Fab") (width 0.1))
+    (fp_circle (center 1.27 0) (end 2.77 0) (layer "F.Fab") (width 0.1) (fill none))
+    (pad "1" thru_hole rect locked (at 0 0) (size 1.8 1.8) (drill 0.9) (layers *.Cu *.Mask)
+      (net 1 "GND"))
+    (pad "2" thru_hole circle locked (at 2.54 0) (size 1.8 1.8) (drill 0.9) (layers *.Cu *.Mask)
+      (net 2 "Pin0"))
+    (model "${KISYS3DMOD}/LED_THT.3dshapes/LED_D3.0mm.wrl"
+      (offset (xyz 0 0 0))
       (scale (xyz 1 1 1))
       (rotate (xyz 0 0 0))
     )
   )
-  (module TestPoint:TestPoint_Pad_D1.5mm (layer B.Cu)
+  (footprint "TestPoint:TestPoint_Pad_D1.5mm" (layer "B.Cu")
     (at 1.27 -2.54)
     (descr "SMD pad as test Point, diameter 1.5mm")
     (tags "test point SMD pad")
-    (attr virtual)
-    (fp_text reference TP1 (at 0 1.648) (layer B.SilkS) hide
+    (attr exclude_from_pos_files exclude_from_bom)
+    (fp_text reference "TP1" (at 0 1.648) (layer "B.SilkS") hide
       (effects (font (size 1 1) (thickness 0.15)) (justify mirror))
     )
-    (fp_text value TestPoint (at 0 -1.75) (layer B.Fab)
+    (fp_text value "TestPoint" (at 0 -1.75) (layer "B.Fab")
       (effects (font (size 1 1) (thickness 0.15)) (justify mirror))
     )
-    (fp_circle (center 0 0) (end 0 -0.95) (layer B.SilkS) (width 0.12))
-    (fp_circle (center 0 0) (end 1.25 0) (layer B.CrtYd) (width 0.05))
-    (fp_text user %R (at 0 1.65) (layer B.Fab)
+    (fp_text user "${REFERENCE}" (at 0 1.65) (layer "B.Fab")
       (effects (font (size 1 1) (thickness 0.15)) (justify mirror))
     )
-    (pad 1 smd circle (at 0 0) (size 1.5 1.5) (layers B.Cu B.Mask)
-      (net 2 Pin0))
+    (fp_circle (center 0 0) (end 0 -0.95) (layer "B.SilkS") (width 0.12) (fill none))
+    (fp_circle (center 0 0) (end 1.25 0) (layer "B.CrtYd") (width 0.05) (fill none))
+    (pad "1" smd circle locked (at 0 0) (size 1.5 1.5) (layers "B.Cu" "B.Mask")
+      (net 2 "Pin0"))
   )
-  (gr_text pin (at 0.254 -2.794) (layer B.SilkS)
+  (gr_circle (center 0 0) (end 1.55 0) (layer "Eco1.User") (width 0.12) (fill none))
+  (gr_text "pin" (at 0.254 -2.794) (layer "B.SilkS")
     (effects (font (size 1 1) (thickness 0.15)) (justify left mirror))
   )
-  (segment (start 1.27 0) (end 1.27 -2.54) (width 0.635) (layer B.Cu) (net 2))
-  (gr_circle (center 0 0) (end 1.55 0) (layer Eco1.User) (width 0.12))
+  (segment (start 1.27 0) (end 1.27 -2.54) (width 0.635) (layer "B.Cu") (net 2))
 )
