File: boards/kivu12/kivu12.cvpitch.kicad_sch (KiCad schematic)
At the start: 14 parts, among them U9 TL072

Commit message: Use shift register instead of multiplexer
Parts:
- C11, C12: DistLink https://www.digikey.de/product-detail/en/avx-corporation/06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 -> https://www.digikey.de/en/products/detail/kyocera-avx/06033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
Changed lines of the file:
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@@
       (effects (font (size 1.27 1.27)) hide)
     )
-    (property "DistLink" "https://www.digikey.de/product-detail/en/avx-corporation/06033C104KAT4A/478-7018-1-ND/3247565" (id 9) (at 198.12 68.58 0)
+    (property "DistLink" "https://www.digikey.de/en/products/detail/kyocera-avx/06033C104KAT4A/3247517" (id 9) (at 198.12 68.58 0)
       (effects (font (size 1.27 1.27)) hide)
     )
@@
       (effects (font (size 1.27 1.27)) hide)
     )
-    (property "DistLink" "https://www.digikey.de/product-detail/en/avx-corporation/06033C104KAT4A/478-7018-1-ND/3247565" (id 9) (at 198.12 81.28 0)
+    (property "DistLink" "https://www.digikey.de/en/products/detail/kyocera-avx/06033C104KAT4A/3247517" (id 9) (at 198.12 81.28 0)
       (effects (font (size 1.27 1.27)) hide)
     )

Commit message: Add support for jlcpcb pcba service
Parts:
- C11, C12: JlcPcbPartNumber (none) -> C14663; Package (none) -> 0603
- C13: JlcPcbPartNumber (none) -> C15849; Package (none) -> 0603
- D22: JlcPcbPartNumber (none) -> C129967; Package (none) -> SOT-23; ReelRotation (none) -> 180
- R68, R69, R72, R73, R81, R82: JlcPcbPartNumber (none) -> C25803; Package (none) -> 0603
- R76: JlcPcbPartNumber (none) -> C23046; Package (none) -> 0603
- U9: JlcPcbPartNumber (none) -> C67473; Package (none) -> SOIC-8; ReelRotation (none) -> 90
- U9: Device (none) -> Op Amp; Dist (none) -> Digikey; DistLink (none) -> https://www.digikey.de/product-detail/en/texas-instruments/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; DistPartNumber (none) -> 296-1282-1-ND; JlcPcbPartNumber (none) -> C67473; Package (none) -> SOIC-8; Place (none) -> Yes; ReelRotation (none) -> 90
Changed lines of the file:
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@@
+      (effects (font (size 1.27 1.27)) hide)
+    )
+    (property "Package" "SOIC-8" (id 10) (at 97.79 78.74 0)
+      (effects (font (size 1.27 1.27)) hide)
+    )
+    (property "JlcPcbPartNumber" "C67473" (id 11) (at 97.79 78.74 0)
+      (effects (font (size 1.27 1.27)) hide)
+    )
+    (property "ReelRotation" "90" (id 12) (at 97.79 78.74 0)
       (effects (font (size 1.27 1.27)) hide)
     )
@@
       (effects (font (size 1.27 1.27)) hide)
     )
+    (property "Device" "Op Amp" (id 4) (at 97.79 121.92 0)
+      (effects (font (size 1.27 1.27)) hide)
+    )
+    (property "Description" "IC OPAMP JFET 2 CIRCUIT 8SOIC" (id 5) (at 97.79 121.92 0)
+      (effects (font (size 1.27 1.27)) hide)
+    )
+    (property "Place" "Yes" (id 6) (at 97.79 121.92 0)
+      (effects (font (size 1.27 1.27)) hide)
+    )
+    (property "Dist" "Digikey" (id 7) (at 97.79 121.92 0)
+      (effects (font (size 1.27 1.27)) hide)
+    )
+    (property "DistPartNumber" "296-1282-1-ND" (id 8) (at 97.79 121.92 0)
+      (effects (font (size 1.27 1.27)) hide)
+    )
+    (property "DistLink" "https://www.digikey.de/product-detail/en/texas-instruments/TL072CDR/296-1282-1-ND/404930" (id 9) (at 97.79 121.92 0)
+      (effects (font (size 1.27 1.27)) hide)
+    )
+    (property "Package" "SOIC-8" (id 10) (at 97.79 121.92 0)
+      (effects (font (size 1.27 1.27)) hide)
+    )
+    (property "JlcPcbPartNumber" "C67473" (id 11) (at 97.79 121.92 0)
+      (effects (font (size 1.27 1.27)) hide)
+    )
+    (property "ReelRotation" "90" (id 12) (at 97.79 121.92 0)
+      (effects (font (size 1.27 1.27)) hide)
+    )
     (pin "1")
     (pin "2")
@@
       (effects (font (size 1.27 1.27)) hide)
     )
+    (property "Device" "Op Amp" (id 4) (at 187.96 74.93 0)
+      (effects (font (size 1.27 1.27)) hide)
+    )
+    (property "Description" "IC OPAMP JFET 2 CIRCUIT 8SOIC" (id 5) (at 187.96 74.93 0)
+      (effects (font (size 1.27 1.27)) hide)
+    )
+    (property "Place" "Yes" (id 6) (at 187.96 74.93 0)
+      (effects (font (size 1.27 1.27)) hide)
+    )
+    (property "Dist" "Digikey" (id 7) (at 187.96 74.93 0)
+      (effects (font (size 1.27 1.27)) hide)
+    )
+    (property "DistPartNumber" "296-1282-1-ND" (id 8) (at 187.96 74.93 0)
+      (effects (font (size 1.27 1.27)) hide)
+    )
+    (property "DistLink" "https://www.digikey.de/product-detail/en/texas-instruments/TL072CDR/296-1282-1-ND/404930" (id 9) (at 187.96 74.93 0)
+      (effects (font (size 1.27 1.27)) hide)
+    )
+    (property "Package" "SOIC-8" (id 10) (at 187.96 74.93 0)
+      (effects (font (size 1.27 1.27)) hide)
+    )
+    (property "JlcPcbPartNumber" "C67473" (id 11) (at 187.96 74.93 0)
+      (effects (font (size 1.27 1.27)) hide)
+    )
+    (property "ReelRotation" "90" (id 12) (at 187.96 74.93 0)
+      (effects (font (size 1.27 1.27)) hide)
+    )
     (pin "1")
     (pin "2")
@@
       (effects (font (size 1.27 1.27)) hide)
     )
+    (property "Package" "0603" (id 10) (at 198.12 68.58 0)
+      (effects (font (size 1.27 1.27)) hide)
+    )
+    (property "JlcPcbPartNumber" "C14663" (id 11) (at 198.12 68.58 0)
+      (effects (font (size 1.27 1.27)) hide)
+    )
     (pin "1")
     (pin "2")
@@
     )
     (property "DistLink" "https://www.digikey.de/en/products/detail/kyocera-avx/06033C104KAT4A/3247517" (id 9) (at 198.12 81.28 0)
+      (effects (font (size 1.27 1.27)) hide)
+    )
+    (property "Package" "0603" (id 10) (at 198.12 81.28 0)
+      (effects (font (size 1.27 1.27)) hide)
+    )
+    (property "JlcPcbPartNumber" "C14663" (id 11) (at 198.12 81.28 0)
       (effects (font (size 1.27 1.27)) hide)
     )
@@
       (effects (font (size 1.27 1.27)) hide)
     )
+    (property "Package" "0603" (id 10) (at 179.07 123.19 0)
+      (effects (font (size 1.27 1.27)) hide)
+    )
+    (property "JlcPcbPartNumber" "C23046" (id 11) (at 179.07 123.19 0)
+      (effects (font (size 1.27 1.27)) hide)
+    )
     (pin "1")
     (pin "2")
@@
     )
     (property "DistLink" "https://www.digikey.de/product-detail/en/texas-instruments/LM4040BIM3-5-0-NOPB/LM4040BIM3-5-0-NOPBCT-ND/212696" (id 9) (at 185.42 127 0)
+      (effects (font (size 1.27 1.27)) hide)
+    )
+    (property "Package" "SOT-23" (id 10) (at 185.42 127 0)
+      (effects (font (size 1.27 1.27)) hide)
+    )
+    (property "JlcPcbPartNumber" "C129967" (id 11) (at 185.42 127 0)
+      (effects (font (size 1.27 1.27)) hide)
+    )
+    (property "ReelRotation" "180" (id 12) (at 185.42 127 0)
       (effects (font (size 1.27 1.27)) hide)
     )
@@
       (effects (font (size 1.27 1.27)) hide)
     )
+    (property "Package" "0603" (id 10) (at 205.74 127 0)
+      (effects (font (size 1.27 1.27)) hide)
+    )
+    (property "JlcPcbPartNumber" "C15849" (id 11) (at 205.74 127 0)
+      (effects (font (size 1.27 1.27)) hide)
+    )
     (pin "1")
     (pin "2")
@@
       (effects (font (size 1.27 1.27)) hide)
     )
+    (property "Package" "0603" (id 10) (at 76.2 76.2 0)
+      (effects (font (size 1.27 1.27)) hide)
+    )
+    (property "JlcPcbPartNumber" "C25803" (id 11) (at 76.2 76.2 0)
+      (effects (font (size 1.27 1.27)) hide)
+    )
     (pin "1")
     (pin "2")
@@
       (effects (font (size 1.27 1.27)) hide)
     )
+    (property "Package" "0603" (id 10) (at 76.2 67.31 0)
+      (effects (font (size 1.27 1.27)) hide)
+    )
+    (property "JlcPcbPartNumber" "C25803" (id 11) (at 76.2 67.31 0)
+      (effects (font (size 1.27 1.27)) hide)
+    )
     (pin "1")
     (pin "2")
@@
       (effects (font (size 1.27 1.27)) hide)
     )
+    (property "Package" "0603" (id 10) (at 76.2 119.38 0)
+      (effects (font (size 1.27 1.27)) hide)
+    )
+    (property "JlcPcbPartNumber" "C25803" (id 11) (at 76.2 119.38 0)
+      (effects (font (size 1.27 1.27)) hide)
+    )
     (pin "1")
     (pin "2")
@@
       (effects (font (size 1.27 1.27)) hide)
     )
+    (property "Package" "0603" (id 10) (at 76.2 110.49 0)
+      (effects (font (size 1.27 1.27)) hide)
+    )
+    (property "JlcPcbPartNumber" "C25803" (id 11) (at 76.2 110.49 0)
+      (effects (font (size 1.27 1.27)) hide)
+    )
     (pin "1")
     (pin "2")
@@
       (effects (font (size 1.27 1.27)) hide)
     )
+    (property "Package" "0603" (id 10) (at 96.52 69.85 0)
+      (effects (font (size 1.27 1.27)) hide)
+    )
+    (property "JlcPcbPartNumber" "C25803" (id 11) (at 96.52 69.85 0)
+      (effects (font (size 1.27 1.27)) hide)
+    )
     (pin "1")
     (pin "2")
@@
       (effects (font (size 1.27 1.27)) hide)
     )
+    (property "Package" "0603" (id 10) (at 96.52 113.03 0)
+      (effects (font (size 1.27 1.27)) hide)
+    )
+    (property "JlcPcbPartNumber" "C25803" (id 11) (at 96.52 113.03 0)
+      (effects (font (size 1.27 1.27)) hide)
+    )
