File: build-system/erbui/generators/front_pcb/thonk.pj398sm.manual/thonk.pj398sm.manual.kicad_pcb (KiCad board)
At the start: 2 copper layers, 1 part, among them J1 IN

Commit message: Wip
Other:
- net class Default removed
Changed lines of the file:
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@@
-(kicad_pcb (version 20171130) (host pcbnew "(5.1.9-0-10_14)")
+(kicad_pcb (version 20211014) (generator pcbnew)
   (general
     (thickness 1.6)
-    (drawings 0)
-    (tracks 0)
-    (zones 0)
-    (modules 1)
-    (nets 4)
   )
-  (page A4)
+  (paper "A4")
   (layers
-    (0 F.Cu signal)
-    (31 B.Cu signal)
-    (32 B.Adhes user)
-    (33 F.Adhes user)
-    (34 B.Paste user)
-    (35 F.Paste user)
-    (36 B.SilkS user)
-    (37 F.SilkS user)
-    (38 B.Mask user)
-    (39 F.Mask user)
-    (40 Dwgs.User user)
-    (41 Cmts.User user)
-    (42 Eco1.User user)
-    (43 Eco2.User user)
-    (44 Edge.Cuts user)
-    (45 Margin user)
-    (46 B.CrtYd user hide)
-    (47 F.CrtYd user hide)
-    (48 B.Fab user hide)
-    (49 F.Fab user hide)
+    (0 "F.Cu" signal)
+    (31 "B.Cu" signal)
+    (32 "B.Adhes" user "B.Adhesive")
+    (33 "F.Adhes" user "F.Adhesive")
+    (34 "B.Paste" user)
+    (35 "F.Paste" user)
+    (36 "B.SilkS" user "B.Silkscreen")
+    (37 "F.SilkS" user "F.Silkscreen")
+    (38 "B.Mask" user)
+    (39 "F.Mask" user)
+    (40 "Dwgs.User" user "User.Drawings")
+    (41 "Cmts.User" user "User.Comments")
+    (42 "Eco1.User" user "User.Eco1")
+    (43 "Eco2.User" user "User.Eco2")
+    (44 "Edge.Cuts" user)
+    (45 "Margin" user)
+    (46 "B.CrtYd" user "B.Courtyard")
+    (47 "F.CrtYd" user "F.Courtyard")
+    (48 "B.Fab" user)
+    (49 "F.Fab" user)
   )
   (setup
-    (last_trace_width 0.1524)
-    (user_trace_width 0.1524)
-    (user_trace_width 0.254)
-    (user_trace_width 0.4064)
-    (user_trace_width 0.635)
-    (trace_clearance 0.1524)
-    (zone_clearance 0.508)
-    (zone_45_only no)
-    (trace_min 0.1524)
-    (via_size 0.6858)
-    (via_drill 0.3048)
-    (via_min_size 0.6858)
-    (via_min_drill 0.3048)
-    (uvia_size 0.3048)
-    (uvia_drill 0.1524)
-    (uvias_allowed no)
-    (uvia_min_size 0.2)
-    (uvia_min_drill 0.1)
-    (edge_width 0.15)
-    (segment_width 0.2)
-    (pcb_text_width 0.3)
-    (pcb_text_size 1.5 1.5)
-    (mod_edge_width 0.15)
-    (mod_text_size 1 1)
-    (mod_text_width 0.15)
-    (pad_size 2 1.3)
-    (pad_drill 1.3)
     (pad_to_mask_clearance 0.2)
-    (aux_axis_origin 0 0)
-    (visible_elements FFFFFF7F)
     (pcbplotparams
-      (layerselection 0x010fc_ffffffff)
+      (layerselection 0x00010fc_ffffffff)
+      (disableapertmacros false)
       (usegerberextensions false)
       (usegerberattributes false)
       (usegerberadvancedattributes false)
       (creategerberjobfile false)
+      (svguseinch false)
+      (svgprecision 6)
       (excludeedgelayer true)
-      (linewidth 0.100000)
       (plotframeref false)
       (viasonmask false)
@@
       (hpglpenspeed 20)
       (hpglpendiameter 15.000000)
+      (dxfpolygonmode true)
+      (dxfimperialunits true)
+      (dxfusepcbnewfont true)
       (psnegative false)
       (psa4output false)
@@
       (plotvalue true)
       (plotinvisibletext false)
-      (padsonsilk false)
+      (sketchpadsonfab false)
       (subtractmaskfromsilk false)
       (outputformat 1)
@@
       (drillshape 1)
       (scaleselection 1)
-      (outputdirectory ""))
+      (outputdirectory "")
+    )
   )
   (net 0 "")
-  (net 1 GND)
-  (net 2 Pin0)
-  (net 3 Cascade0)
-  (net_class Default "This is the default net class."
-    (clearance 0.1524)
-    (trace_width 0.1524)
-    (via_dia 0.6858)
-    (via_drill 0.3048)
-    (uvia_dia 0.3048)
-    (uvia_drill 0.1524)
-    (diff_pair_width 0.1524)
-    (diff_pair_gap 0.1524)
-    (add_net Cascade0)
-    (add_net GND)
-    (add_net Pin0)
-  )
-  (module Connector_Thonk:ThonkiconnJack locked (layer F.Cu)
+  (net 1 "GND")
+  (net 2 "Pin0")
+  (net 3 "Cascade0")
+  (footprint "Connector_Thonk:ThonkiconnJack" locked (layer "F.Cu")
     (at 0 0)
-    (fp_text reference J1 (at -2.84 -4.94) (layer F.SilkS)
+    (attr through_hole)
+    (fp_text reference "J1" (at -2.84 -4.94) (layer "F.SilkS")
       (effects (font (size 1 1) (thickness 0.15)))
     )
-    (fp_text value IN (at 0 9.3) (layer F.Fab)
+    (fp_text value "IN" (at 0 9.3) (layer "F.Fab")
       (effects (font (size 1 1) (thickness 0.15)))
     )
-    (fp_line (start -4.5 4.5) (end 4.5 4.5) (layer F.SilkS) (width 0.15))
-    (fp_line (start 4.5 -6) (end 4.5 4.5) (layer F.SilkS) (width 0.15))
-    (fp_line (start -4.5 -6) (end -4.5 4.5) (layer F.SilkS) (width 0.15))
-    (fp_line (start -4.5 -6) (end 4.5 -6) (layer F.SilkS) (width 0.15))
-    (fp_circle (center 0 0) (end 1.8 0) (layer F.SilkS) (width 0.15))
-    (pad "" np_thru_hole circle (at 0 0) (size 2.5 2.5) (drill 2.5) (layers *.Cu *.Mask))
-    (pad T thru_hole oval (at 0 -4.92) (size 2.2 1.2) (drill oval 1.5 0.5) (layers *.Cu *.Mask)
-      (net 2 Pin0))
-    (pad TN thru_hole oval (at 0 3.38) (size 2.2 1.3) (drill oval 1.5 0.6) (layers *.Cu *.Mask)
-      (net 3 Cascade0))
-    (pad S thru_hole oval (at 0 6.48) (size 2 1.3) (drill oval 1.3 0.6) (layers *.Cu *.Mask)
-      (net 1 GND))
+    (fp_line (start -4.5 4.5) (end 4.5 4.5) (layer "F.SilkS") (width 0.15))
+    (fp_line (start -4.5 -6) (end 4.5 -6) (layer "F.SilkS") (width 0.15))
+    (fp_line (start 4.5 -6) (end 4.5 4.5) (layer "F.SilkS") (width 0.15))
+    (fp_line (start -4.5 -6) (end -4.5 4.5) (layer "F.SilkS") (width 0.15))
+    (fp_circle (center 0 0) (end 1.8 0) (layer "F.SilkS") (width 0.15) (fill none))
+    (pad "" np_thru_hole circle locked (at 0 0) (size 2.5 2.5) (drill 2.5) (layers *.Cu *.Mask))
+    (pad "S" thru_hole oval locked (at 0 6.48) (size 2 1.3) (drill oval 1.3 0.6) (layers *.Cu *.Mask)
+      (net 1 "GND"))
+    (pad "T" thru_hole oval locked (at 0 -4.92) (size 2.2 1.2) (drill oval 1.5 0.5) (layers *.Cu *.Mask)
+      (net 2 "Pin0"))
+    (pad "TN" thru_hole oval locked (at 0 3.38) (size 2.2 1.3) (drill oval 1.5 0.6) (layers *.Cu *.Mask)
+      (net 3 "Cascade0"))
   )
-  (gr_circle (center 0 0) (end 3.25 0) (layer Eco1.User) (width 0.12))
+  (gr_circle (center 0 0) (end 3.25 0) (layer "Eco1.User") (width 0.12) (fill none))
 )

Commit message: Replace cascade feature with normalling feature
Connections:
- net Cascade0 renamed Normalling0
Changed lines of the file:
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@@
   (net 1 "GND")
   (net 2 "Pin0")
-  (net 3 "Cascade0")
+  (net 3 "Normalling0")
   (footprint "Connector_Thonk:ThonkiconnJack" locked (layer "F.Cu")
     (at 0 0)
+    (property "Description" "Thonkiconn – 3.5mm Jack Sockets")
+    (property "Device" "Jack Connector")
+    (property "Dist" "Thonk")
+    (property "DistLink" "https://www.thonk.co.uk/shop/thonkiconn/")
+    (property "DistPartNumber" "PJ398SM")
+    (property "Place" "No")
+    (property "Sheetfile" "thonk.pj398sm.manual.kicad_sch")
+    (property "Sheetname" "")
     (attr through_hole)
     (fp_text reference "J1" (at -2.84 -4.94) (layer "F.SilkS")
@@
     (pad "" np_thru_hole circle locked (at 0 0) (size 2.5 2.5) (drill 2.5) (layers *.Cu *.Mask))
     (pad "S" thru_hole oval locked (at 0 6.48) (size 2 1.3) (drill oval 1.3 0.6) (layers *.Cu *.Mask)
-      (net 1 "GND"))
+      (net 1 "GND") (pintype "passive"))
     (pad "T" thru_hole oval locked (at 0 -4.92) (size 2.2 1.2) (drill oval 1.5 0.5) (layers *.Cu *.Mask)
-      (net 2 "Pin0"))
+      (net 2 "Pin0") (pintype "passive"))
     (pad "TN" thru_hole oval locked (at 0 3.38) (size 2.2 1.3) (drill oval 1.5 0.6) (layers *.Cu *.Mask)
-      (net 3 "Cascade0"))
+      (net 3 "Normalling0") (pintype "passive"))
   )
   (gr_circle (center 0 0) (end 3.25 0) (layer "Eco1.User") (width 0.12) (fill none))
