File: build-system/erbui/generators/front_pcb/thonk.pj398sm.wire.npr/thonk.pj398sm.wire.npr.kicad_pcb (KiCad board)
At the start: 2 copper layers, 5 parts, among them J1 IN

Commit message: Use npr reference instead of normalling reference
Other:
- board text added: "NPR"
- board text removed: "normalling_from"
Changed lines of the file:
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@@
     (effects (font (size 1 1) (thickness 0.15)) (justify left mirror))
   )
-  (gr_text "normalling_from" (at -1.4 0.1) (layer "B.SilkS")
+  (gr_text "NPR" (at -1.4 0.1) (layer "B.SilkS")
     (effects (font (size 1 1) (thickness 0.15)) (justify left mirror))
   )
