File: build-system/erbui/generators/front_pcb/ck.d6r.black.wire/ck.d6r.black.wire.kicad_sch (KiCad schematic)
At the start: 2 parts, among them SW1 SW_Push_Dual

Commit message: Remove deprecated simulator class field from schematic files
Parts:
- SW1: Simulator erb::Ckd6r -> (none)
Changed lines of the file:
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@@
-      (effects (font (size 1.27 1.27)) hide)
-    )
-    (property "Simulator" "erb::Ckd6r" (id 10) (at 119.38 134.62 0)
       (effects (font (size 1.27 1.27)) hide)
     )
