File: build-system/erbui/generators/front_pcb/led.3mm.green.wire/led.3mm.green.wire.kicad_sch (KiCad schematic)
At the start: 2 parts

Commit message: Remove deprecated simulator class field from schematic files
Parts:
- D1: Simulator erb::Led3mm <GreenLight> -> (none)
Changed lines of the file:
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@@
-      (effects (font (size 1.27 1.27)) hide)
-    )
-    (property "Simulator" "erb::Led3mm <GreenLight>" (id 10) (at 129.54 128.27 0)
       (effects (font (size 1.27 1.27)) hide)
     )
