File: build-system/erbui/generators/front_pcb/thonk.pj398sm.knurled/thonk.pj398sm.knurled.kicad_sch (KiCad schematic)
At the start: 1 part

Commit message: Remove deprecated simulator class field from schematic files
Parts:
- H1: Simulator erb::ThonkPj398SmKnurled -> (none)
Changed lines of the file:
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@@
-      (effects (font (size 1.27 1.27)) hide)
-    )
-    (property "Simulator" "erb::ThonkPj398SmKnurled" (id 10) (at 110.49 74.93 90)
       (effects (font (size 1.27 1.27)) hide)
     )
