File: samples/custom/manufacturer/rogan.6ps/rogan.6ps.kicad_sch (KiCad schematic)
At the start: 1 part

Commit message: Update samples
Parts:
- H1: Simulator erb::AlphaPot <erb::Rogan6Ps> -> (none)
Changed lines of the file:
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@@
-      (effects (font (size 1.27 1.27)) hide)
-    )
-    (property "Simulator" "erb::AlphaPot <erb::Rogan6Ps>" (id 7) (at 110.49 74.93 90)
       (effects (font (size 1.27 1.27)) hide)
     )
