File: build-system/erbui/generators/front_pcb/dailywell.2ms3.wire/dailywell.2ms3.wire.kicad_sch (KiCad schematic)
At the start: 3 parts, among them SW1 SW_SPDT

Commit message: Remove deprecated simulator class field from schematic files
Parts:
- SW1: Simulator erb::Dailywell2Ms3 -> (none)
Changed lines of the file:
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@@
-      (effects (font (size 1.27 1.27)) hide)
-    )
-    (property "Simulator" "erb::Dailywell2Ms3" (id 10) (at 127 119.38 0)
       (effects (font (size 1.27 1.27)) hide)
     )

Commit message: Move switch number positions to manufacturer control definition
Parts:
- SW1: NbrPositions 3 -> (none)
Changed lines of the file:
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@@
-      (effects (font (size 1.27 1.27)) hide)
-    )
-    (property "NbrPositions" "3" (id 11) (at 127 119.38 0)
       (effects (font (size 1.27 1.27)) hide)
     )
